File: PCB Files/Circuit-Teensy32/OpeNITHM.kicad_pcb (KiCad board)
At the start: 2 copper layers, 100 x 45.3 mm, 26 parts, among them J1 Conn_01x14, J2 Conn_01x14, J3 Conn_02x07_Odd_Even, J7 Conn_02x12_Odd_Even, J8 Conn_02x12_Odd_Even, J9 Conn_01x05, U1 74HC4051, U2 74HC4051, U3 74HC4051, U4 74HC4051

Commit message: Fixed RGB labeling on back silkscreen
Other:
- board text removed: "RGB C0"
